File: unmechanical-sweepish/unmechanical-sweepish-r.kicad_sch (KiCad schematic)
At the start: 82 parts, among them J3 M, Q1 AO3400A, U11 OPA340NA, U5 74HC4051

Commit message: update to kicad 8 model paths
Parts:
- J4: renamed from J?; footprint PCM_marbastlib-xp-various:CON_HytePro_M411P_Receptacle_1x04-P2.20mm_Horizontal_FlushMount -> PCM_marbastlib-various:CON_HytePro_M411P_Receptacle_1x04-P2.20mm_Horizontal_FlushMount
- L2: value BLM15PX121SN1D -> BLM15PX121SN1D
- gave numbers to parts that had none: 22
- renumbered C16 to C22, EC1 to EC19, EC2 to EC20, EC3 to EC21, EC4 to EC22, EC5 to EC23, EC6 to EC24, EC7 to EC25, EC8 to EC26, EC9 to EC27, EC10 to EC28, EC11 to EC29, EC12 to EC30, EC13 to EC31, EC14 to EC32, EC15 to EC33, EC16 to EC34, EC17 to EC35, EC18 to EC36, F1 to F2, H1 to H5, H2 to H6, H3 to H7, H4 to H8, J3 to J6, Q1 to Q2, R18 to R23, R18 to R24, R10 to R25, R18 to R26, R17 to R27, R3 to R30, R4 to R31, R5 to R32, R6 to R33, R7 to R34, R9 to R35, R10 to R36, R11 to R37, R12 to R39, R13 to R40, R14 to R41, R15 to R42, U5 to U10, U11 to U9
